Commit message: first

File: robot/TOE_dog/urdf/dog.urdf (robot description, URDF)
Before this commit: robot TOE_dog, 17 links, 16 joints
Links:
- link FL_calf: geometry collision box size=0.16 0.0245 0.04; visual mesh filename=package://urdf_tutorial/meshes/TOE_calf.STL
- link FL_foot: geometry collision sphere radius=0.022; visual mesh filename=package://urdf_tutorial/meshes/TOE_foot.STL
- link FL_hip: geometry collision cylinder length=0.08 radius=0.046; visual mesh filename=package://urdf_tutorial/meshes/TOE_FL_hip.STL
- link FL_thigh: geometry collision box size=0.11 0.0245 0.04; visual mesh filename=package://urdf_tutorial/meshes/TOE_thigh.STL
- link FR_calf: geometry collision box size=0.16 0.0245 0.04; visual mesh filename=package://urdf_tutorial/meshes/TOE_calf.STL
- link FR_foot: geometry collision sphere radius=0.022; visual mesh filename=package://urdf_tutorial/meshes/TOE_foot.STL
- link FR_hip: geometry collision cylinder length=0.08 radius=0.046; visual mesh filename=package://urdf_tutorial/meshes/TOE_FR_hip.STL
- link FR_thigh: geometry collision box size=0.11 0.0245 0.04; visual mesh filename=package://urdf_tutorial/meshes/TOE_R_thigh.STL
- link RL_calf: geometry collision box size=0.16 0.0245 0.04; visual mesh filename=package://urdf_tutorial/meshes/TOE_calf.STL
- link RL_foot: geometry collision sphere radius=0.022; visual mesh filename=package://urdf_tutorial/meshes/TOE_foot.STL
- link RL_hip: geometry collision cylinder length=0.08 radius=0.046; visual mesh filename=package://urdf_tutorial/meshes/TOE_RL_hip.STL
- link RL_thigh: geometry collision box size=0.11 0.0245 0.04; visual mesh filename=package://urdf_tutorial/meshes/TOE_thigh.STL
- link RR_calf: geometry collision box size=0.16 0.0245 0.04; visual mesh filename=package://urdf_tutorial/meshes/TOE_calf.STL
- link RR_foot: geometry collision sphere radius=0.022; visual mesh filename=package://urdf_tutorial/meshes/TOE_foot.STL
- link RR_hip: geometry collision cylinder length=0.08 radius=0.046; visual mesh filename=package://urdf_tutorial/meshes/TOE_RR_hip.STL
- link RR_thigh: geometry collision box size=0.11 0.0245 0.04; visual mesh filename=package://urdf_tutorial/meshes/TOE_R_thigh.STL
- link base: mass 4.991 -> 5.1234705; geometry collision box size=0.27 0.15 0.114; visual mesh filename=package://urdf_tutorial/meshes/TOE_base.STL
Joints:
- joint FL_calf_joint: limit lower=-2.6 upper=-1 effort=35 velocity=20 -> lower=-2.6 upper=-0.15 effort=35 velocity=20
- joint FL_foot_joint: origin xyz=0.0 0 -0.20051 rpy=0 -0.0012583 0 -> xyz=0 0 -0.20051 rpy=0 -0.0012583 0
- joint FR_calf_joint: limit lower=-2.6 upper=-1 effort=35 velocity=20 -> lower=-2.6 upper=-0.15 effort=35 velocity=20
- joint RL_calf_joint: limit lower=-2.6 upper=-1 effort=35 velocity=20 -> lower=-2.6 upper=-0.15 effort=35 velocity=20
- joint RR_calf_joint: limit lower=-2.6 upper=-1 effort=35 velocity=20 -> lower=-2.6 upper=-0.15 effort=35 velocity=20

Commit message: first

File: robot/TOE_dog/urdf/dog.urdf (robot description, URDF)
Before this commit: robot TOE_dog, 17 links, 16 joints
Links:
- link FL_calf: geometry collision box size=0.16 0.0245 0.04; visual mesh filename=../assets/TOE_calf.STL
- link FL_foot: geometry collision sphere radius=0.022; visual mesh filename=../assets/TOE_foot.STL
- link FL_hip: geometry collision cylinder length=0.08 radius=0.046; visual mesh filename=../assets/TOE_FL_hip.STL
- link FL_thigh: geometry collision box size=0.11 0.0245 0.04; visual mesh filename=../assets/TOE_L_thigh.STL
- link FR_calf: geometry collision box size=0.16 0.0245 0.04; visual mesh filename=../assets/TOE_calf.STL
- link FR_foot: geometry collision sphere radius=0.022; visual mesh filename=../assets/TOE_foot.STL
- link FR_hip: geometry collision cylinder length=0.08 radius=0.046; visual mesh filename=../assets/TOE_FR_hip.STL
- link FR_thigh: geometry collision box size=0.11 0.0245 0.04; visual mesh filename=../assets/TOE_R_thigh.STL
- link RL_calf: geometry collision box size=0.16 0.0245 0.04; visual mesh filename=../assets/TOE_calf.STL
- link RL_foot: geometry collision sphere radius=0.022; visual mesh filename=../assets/TOE_foot.STL
- link RL_hip: geometry collision cylinder length=0.08 radius=0.046; visual mesh filename=../assets/TOE_RL_hip.STL
- link RL_thigh: geometry collision box size=0.11 0.0245 0.04; visual mesh filename=../assets/TOE_L_thigh.STL
- link RR_calf: geometry collision box size=0.16 0.0245 0.04; visual mesh filename=../assets/TOE_calf.STL
- link RR_foot: geometry collision sphere radius=0.022; visual mesh filename=../assets/TOE_foot.STL
- link RR_hip: geometry collision cylinder length=0.08 radius=0.046; visual mesh filename=../assets/TOE_RR_hip.STL
- link RR_thigh: geometry collision box size=0.11 0.0245 0.04; visual mesh filename=../assets/TOE_R_thigh.STL
- link base: geometry collision box size=0.27 0.15 0.114; visual mesh filename=../assets/TOE_base.STL

File: robot/TOE_dog/urdf/dog_ros.urdf (robot description, URDF)
Before this commit: robot TOE_dog, 17 links, 16 joints
Links:
- link base: mass 4.991 -> 5.1234705
Joints:
- joint FL_calf_joint: limit lower=-2.6 upper=-1 effort=35 velocity=20 -> lower=-2.6 upper=-0.15 effort=35 velocity=20
- joint FL_foot_joint: origin xyz=0.00081567 0 -0.20051 rpy=0 -0.0012583 0 -> xyz=0 0 -0.20051 rpy=0 -0.0012583 0
- joint FR_calf_joint: limit lower=-2.6 upper=-1 effort=35 velocity=20 -> lower=-2.6 upper=-0.15 effort=35 velocity=20
- joint FR_foot_joint: origin xyz=0.00081567 0 -0.20051 rpy=0 -0.0012583 0 -> xyz=0 0 -0.20051 rpy=0 -0.0012583 0
- joint RL_calf_joint: limit lower=-2.6 upper=-1 effort=35 velocity=20 -> lower=-2.6 upper=-0.15 effort=35 velocity=20
- joint RL_foot_joint: origin xyz=0.00081567 0 -0.20051 rpy=0 -0.0012583 0 -> xyz=0 0 -0.20051 rpy=0 -0.0012583 0
- joint RR_calf_joint: limit lower=-2.6 upper=-1 effort=35 velocity=20 -> lower=-2.6 upper=-0.15 effort=35 velocity=20
- joint RR_foot_joint: origin xyz=0.00081567 0 -0.20051 rpy=0 -0.0012583 0 -> xyz=0 0 -0.20051 rpy=0 -0.0012583 0

Commit message: first

File: robot/TOE_dog/urdf/dog.urdf (robot description, URDF)
Before this commit: robot TOE_dog, 17 links, 16 joints
Links:
- added link imu, mass 0
- link FL_calf: geometry collision box size=0.16 0.0245 0.04; visual mesh filename=../assets/meshes/TOE_calf.STL
- link FL_foot: mass 0.03219067 -> 0.04; geometry collision sphere radius=0.022; visual mesh filename=../assets/meshes/TOE_foot.STL
- link FL_hip: geometry collision cylinder length=0.08 radius=0.046; visual mesh filename=../assets/meshes/TOE_FL_hip.STL
- link FL_thigh: geometry collision box size=0.11 0.0245 0.04; visual mesh filename=../assets/meshes/TOE_L_thigh.STL
- link FR_calf: geometry collision box size=0.16 0.0245 0.04; visual mesh filename=../assets/meshes/TOE_calf.STL
- link FR_foot: mass 0.03219067 -> 0.04; geometry collision sphere radius=0.022; visual mesh filename=../assets/meshes/TOE_foot.STL
- link FR_hip: geometry collision cylinder length=0.08 radius=0.046; visual mesh filename=../assets/meshes/TOE_FR_hip.STL
- link FR_thigh: geometry collision box size=0.11 0.0245 0.04; visual mesh filename=../assets/meshes/TOE_R_thigh.STL
- link RL_calf: geometry collision box size=0.16 0.0245 0.04; visual mesh filename=../assets/meshes/TOE_calf.STL
- link RL_foot: mass 0.03219067 -> 0.04; geometry collision sphere radius=0.022; visual mesh filename=../assets/meshes/TOE_foot.STL
- link RL_hip: geometry collision cylinder length=0.08 radius=0.046; visual mesh filename=../assets/meshes/TOE_RL_hip.STL
- link RL_thigh: geometry collision box size=0.11 0.0245 0.04; visual mesh filename=../assets/meshes/TOE_L_thigh.STL
- link RR_calf: geometry collision box size=0.16 0.0245 0.04; visual mesh filename=../assets/meshes/TOE_calf.STL
- link RR_foot: mass 0.03219067 -> 0.04; geometry collision sphere radius=0.022; visual mesh filename=../assets/meshes/TOE_foot.STL
- link RR_hip: geometry collision cylinder length=0.08 radius=0.046; visual mesh filename=../assets/meshes/TOE_RR_hip.STL
- link RR_thigh: geometry collision box size=0.11 0.0245 0.04; visual mesh filename=../assets/meshes/TOE_R_thigh.STL
- link base: geometry collision box size=0.27 0.15 0.114; visual mesh filename=../assets/meshes/TOE_base.STL
Joints:
- added joint imu_joint: type fixed, parent base, child imu, origin xyz=0 0 0.05764 rpy=0 0 0, axis 0 0 0

File: robot/TOE_dog/urdf/dog_ros.urdf (robot description, URDF)
Before this commit: robot TOE_dog, 17 links, 16 joints
Links:
- added link imu, mass 0
- link FL_foot: mass 0.03219067 -> 0.04
- link FR_foot: mass 0.03219067 -> 0.04
- link RL_foot: mass 0.03219067 -> 0.04
- link RR_foot: mass 0.03219067 -> 0.04
Joints:
- added joint imu_joint: type fixed, parent base, child imu, origin xyz=0 0 0.05764 rpy=0 0 0, axis 0 0 0

Commit message: fist

File: robot/TOE_dog/urdf/dog.urdf (robot description, URDF)
Before this commit: robot TOE_dog, 18 links, 17 joints
Links:
- added link FL_calflower; collision cylinder length=0.07 radius=0.011
- added link FL_calflower1; collision cylinder length=0.02 radius=0.0125
- added link FR_calflower; collision cylinder length=0.07 radius=0.011
- added link FR_calflower1; collision cylinder length=0.02 radius=0.0125
- added link RL_calflower; collision cylinder length=0.07 radius=0.011
- added link RL_calflower1; collision cylinder length=0.02 radius=0.0125
- added link RR_calflower; collision cylinder length=0.07 radius=0.011
- added link RR_calflower1; collision cylinder length=0.02 radius=0.0125
- link FL_calf: geometry collision cylinder length=0.12 radius=0.010; visual mesh filename=../assets/TOE_calf.STL
- link FL_foot: geometry collision sphere radius=0.022; visual mesh filename=../assets/TOE_foot.STL
- link FL_hip: geometry collision cylinder length=0.08 radius=0.046; visual mesh filename=../assets/TOE_FL_hip.STL
- link FL_thigh: geometry collision box size=0.11 0.0245 0.025; visual mesh filename=../assets/TOE_L_thigh.STL
- link FR_calf: geometry collision cylinder length=0.12 radius=0.010; visual mesh filename=../assets/TOE_calf.STL
- link FR_foot: geometry collision sphere radius=0.022; visual mesh filename=../assets/TOE_foot.STL
- link FR_hip: geometry collision cylinder length=0.08 radius=0.046; visual mesh filename=../assets/TOE_FR_hip.STL
- link FR_thigh: geometry collision box size=0.11 0.0245 0.025; visual mesh filename=../assets/TOE_R_thigh.STL
- link RL_calf: geometry collision cylinder length=0.12 radius=0.010; visual mesh filename=../assets/TOE_calf.STL
- link RL_foot: geometry collision sphere radius=0.022; visual mesh filename=../assets/TOE_foot.STL
- link RL_hip: geometry collision cylinder length=0.08 radius=0.046; visual mesh filename=../assets/TOE_RL_hip.STL
- link RL_thigh: geometry collision box size=0.11 0.0245 0.025; visual mesh filename=../assets/TOE_L_thigh.STL
- link RR_calf: geometry collision cylinder length=0.12 radius=0.010; visual mesh filename=../assets/TOE_calf.STL
- link RR_foot: geometry collision sphere radius=0.022; visual mesh filename=../assets/TOE_foot.STL
- link RR_hip: geometry collision cylinder length=0.08 radius=0.046; visual mesh filename=../assets/TOE_RR_hip.STL
- link RR_thigh: geometry collision box size=0.11 0.0245 0.025; visual mesh filename=../assets/TOE_R_thigh.STL
- link base: geometry collision box size=0.27 0.15 0.114; visual mesh filename=../assets/TOE_base.STL
Joints:
- added joint FL_calflower1_joint: type fixed, parent FL_calflower, child FL_calflower1, origin xyz=-0.002 0 -0.042 rpy=0 0.3 0, axis 0 0 0
- added joint FL_calflower_joint: type fixed, parent FL_calf, child FL_calflower, origin xyz=0.005 0 -0.14 rpy=0 -0.1 0, axis 0 0 0
- added joint FR_calflower1_joint: type fixed, parent FR_calflower, child FR_calflower1, origin xyz=-0.002 0 -0.042 rpy=0 0.3 0, axis 0 0 0
- added joint FR_calflower_joint: type fixed, parent FR_calf, child FR_calflower, origin xyz=0.005 0 -0.14 rpy=0 -0.1 0, axis 0 0 0
- added joint RL_calflower1_joint: type fixed, parent RL_calflower, child RL_calflower1, origin xyz=-0.002 0 -0.042 rpy=0 0.3 0, axis 0 0 0
- added joint RL_calflower_joint: type fixed, parent RL_calf, child RL_calflower, origin xyz=0.005 0 -0.14 rpy=0 -0.1 0, axis 0 0 0
- added joint RR_calflower1_joint: type fixed, parent RR_calflower, child RR_calflower1, origin xyz=-0.002 0 -0.042 rpy=0 0.3 0, axis 0 0 0
- added joint RR_calflower_joint: type fixed, parent RR_calf, child RR_calflower, origin xyz=0.005 0 -0.14 rpy=0 -0.1 0, axis 0 0 0
- joint FL_calf_joint: limit lower=-2.6 upper=-0.15 effort=35 velocity=20 -> lower=-2.3 upper=-0.8 effort=30 velocity=20
- joint FL_foot_joint: origin xyz=0 0 -0.20051 rpy=0 -0.0012583 0 -> xyz=0 0 -0.20051 rpy=0 0 0
- joint FL_hip_joint: limit lower=-1 upper=1 effort=23 velocity=30 -> lower=-1 upper=1 effort=23 velocity=20
- joint FL_thigh_joint: limit lower=-1.5 upper=2.5 effort=23 velocity=30 -> lower=-1.5 upper=2.5 effort=23 velocity=20
- joint FR_calf_joint: limit lower=-2.6 upper=-0.15 effort=35 velocity=20 -> lower=-2.3 upper=-0.8 effort=35 velocity=20
- joint FR_foot_joint: origin xyz=0 0 -0.20051 rpy=0 -0.0012583 0 -> xyz=0 0 -0.20051 rpy=0 0 0
- joint FR_hip_joint: limit lower=-1 upper=1 effort=23 velocity=30 -> lower=-1 upper=1 effort=23 velocity=20
- joint FR_thigh_joint: limit lower=-1.5 upper=2.5 effort=23 velocity=30 -> lower=-1.5 upper=2.5 effort=23 velocity=20
- joint RL_calf_joint: limit lower=-2.6 upper=-0.15 effort=35 velocity=20 -> lower=-2.3 upper=-0.8 effort=35 velocity=20
- joint RL_hip_joint: limit lower=-1 upper=1 effort=23 velocity=30 -> lower=-1 upper=1 effort=23 velocity=20
- joint RL_thigh_joint: limit lower=-1.5 upper=2.5 effort=23 velocity=30 -> lower=-1.5 upper=2.5 effort=23 velocity=20
- joint RR_calf_joint: limit lower=-2.6 upper=-0.15 effort=35 velocity=20 -> lower=-2.3 upper=-0.8 effort=32 velocity=20
- joint RR_foot_joint: axis (none) -> 0 0 0; origin xyz=0 0 -0.20051 rpy=0 -0.0012583 0 -> xyz=0 0 -0.20051 rpy=0 0 0
- joint RR_hip_joint: limit lower=-1 upper=1 effort=23 velocity=30 -> lower=-1 upper=1 effort=23 velocity=20
- joint RR_thigh_joint: limit lower=-1.5 upper=2.5 effort=23 velocity=30 -> lower=-1.5 upper=2.5 effort=23 velocity=20
- joint imu_joint: origin xyz=0 0 0.05764 rpy=0 0 0 -> xyz=0 0 0.0 rpy=0 0 0

File: robot/TOE_dog/urdf/dog_ros.urdf (robot description, URDF)
Before this commit: robot TOE_dog, 18 links, 17 joints
Links:
- added link FL_calflower; collision cylinder length=0.07 radius=0.011
- added link FL_calflower1; collision cylinder length=0.02 radius=0.0125
- added link FR_calflower; collision cylinder length=0.07 radius=0.011
- added link FR_calflower1; collision cylinder length=0.02 radius=0.0125
- added link RL_calflower; collision cylinder length=0.07 radius=0.011
- added link RL_calflower1; collision cylinder length=0.02 radius=0.0125
- added link RR_calflower; collision cylinder length=0.07 radius=0.011
- added link RR_calflower1; collision cylinder length=0.02 radius=0.0125
- link FL_calf: geometry collision cylinder length=0.12 radius=0.010; visual mesh filename=package://urdf_tutorial/meshes/TOE_calf.STL
- link FL_thigh: geometry collision box size=0.11 0.0245 0.025; visual mesh filename=package://urdf_tutorial/meshes/TOE_L_thigh.STL
- link FR_calf: geometry collision cylinder length=0.12 radius=0.010; visual mesh filename=package://urdf_tutorial/meshes/TOE_calf.STL
- link FR_thigh: geometry collision box size=0.11 0.0245 0.025; visual mesh filename=package://urdf_tutorial/meshes/TOE_R_thigh.STL
- link RL_calf: geometry collision cylinder length=0.12 radius=0.010; visual mesh filename=package://urdf_tutorial/meshes/TOE_calf.STL
- link RL_thigh: geometry collision box size=0.11 0.0245 0.025; visual mesh filename=package://urdf_tutorial/meshes/TOE_L_thigh.STL
- link RR_calf: geometry collision cylinder length=0.12 radius=0.010; visual mesh filename=package://urdf_tutorial/meshes/TOE_calf.STL
- link RR_thigh: geometry collision box size=0.11 0.0245 0.025; visual mesh filename=package://urdf_tutorial/meshes/TOE_R_thigh.STL
Joints:
- added joint FL_calflower1_joint: type fixed, parent FL_calflower, child FL_calflower1, origin xyz=-0.002 0 -0.042 rpy=0 0.3 0, axis 0 0 0
- added joint FL_calflower_joint: type fixed, parent FL_calf, child FL_calflower, origin xyz=0.005 0 -0.14 rpy=0 -0.1 0, axis 0 0 0
- added joint FR_calflower1_joint: type fixed, parent FR_calflower, child FR_calflower1, origin xyz=-0.002 0 -0.042 rpy=0 0.3 0, axis 0 0 0
- added joint FR_calflower_joint: type fixed, parent FR_calf, child FR_calflower, origin xyz=0.005 0 -0.14 rpy=0 -0.1 0, axis 0 0 0
- added joint RL_calflower1_joint: type fixed, parent RL_calflower, child RL_calflower1, origin xyz=-0.002 0 -0.042 rpy=0 0.3 0, axis 0 0 0
- added joint RL_calflower_joint: type fixed, parent RL_calf, child RL_calflower, origin xyz=0.005 0 -0.14 rpy=0 -0.1 0, axis 0 0 0
- added joint RR_calflower1_joint: type fixed, parent RR_calflower, child RR_calflower1, origin xyz=-0.002 0 -0.042 rpy=0 0.3 0, axis 0 0 0
- added joint RR_calflower_joint: type fixed, parent RR_calf, child RR_calflower, origin xyz=0.005 0 -0.14 rpy=0 -0.1 0, axis 0 0 0
- joint FL_calf_joint: limit lower=-2.6 upper=-0.15 effort=35 velocity=20 -> lower=-2.3 upper=-0.8 effort=30 velocity=20
- joint FL_foot_joint: origin xyz=0 0 -0.20051 rpy=0 -0.0012583 0 -> xyz=0 0 -0.20051 rpy=0 0 0
- joint FL_hip_joint: limit lower=-1 upper=1 effort=23 velocity=30 -> lower=-1 upper=1 effort=23 velocity=20
- joint FL_thigh_joint: limit lower=-1.5 upper=2.5 effort=23 velocity=30 -> lower=-1.5 upper=2.5 effort=23 velocity=20
- joint FR_calf_joint: limit lower=-2.6 upper=-0.15 effort=35 velocity=20 -> lower=-2.3 upper=-0.8 effort=35 velocity=20
- joint FR_foot_joint: origin xyz=0 0 -0.20051 rpy=0 -0.0012583 0 -> xyz=0 0 -0.20051 rpy=0 0 0
- joint FR_hip_joint: limit lower=-1 upper=1 effort=23 velocity=30 -> lower=-1 upper=1 effort=23 velocity=20
- joint FR_thigh_joint: limit lower=-1.5 upper=2.5 effort=23 velocity=30 -> lower=-1.5 upper=2.5 effort=23 velocity=20
- joint RL_calf_joint: limit lower=-2.6 upper=-0.15 effort=35 velocity=20 -> lower=-2.3 upper=-0.8 effort=35 velocity=20
- joint RL_hip_joint: limit lower=-1 upper=1 effort=23 velocity=30 -> lower=-1 upper=1 effort=23 velocity=20
- joint RL_thigh_joint: limit lower=-1.5 upper=2.5 effort=23 velocity=30 -> lower=-1.5 upper=2.5 effort=23 velocity=20
- joint RR_calf_joint: limit lower=-2.6 upper=-0.15 effort=35 velocity=20 -> lower=-2.3 upper=-0.8 effort=32 velocity=20
- joint RR_foot_joint: axis (none) -> 0 0 0; origin xyz=0 0 -0.20051 rpy=0 -0.0012583 0 -> xyz=0 0 -0.20051 rpy=0 0 0
- joint RR_hip_joint: limit lower=-1 upper=1 effort=23 velocity=30 -> lower=-1 upper=1 effort=23 velocity=20
- joint RR_thigh_joint: limit lower=-1.5 upper=2.5 effort=23 velocity=30 -> lower=-1.5 upper=2.5 effort=23 velocity=20
- joint imu_joint: origin xyz=0 0 0.05764 rpy=0 0 0 -> xyz=0 0 0.0 rpy=0 0 0
